File: Hardware/MyoWare_Power_Shield.brd (EAGLE design)
At the start: 52.1 x 20.8 mm, 14 parts

Commit message: Tweaks to bring up to checklist standards
Parts:
- added FID1, FID2: FIDUCIAL1X2, SparkFun-Aesthetics:FIDUCIAL-1X2
Connections:
- net +VS renamed VCC
Other:
- board text added: "+VS"
- board text added: "0.13" diameter typical"
- board text added: "All units in inches"
- board text added: "GND"
- board text added: "SHLD"

Commit message: Moved power trace to back
Routing:
- net VCC: track 55.3 -> 52.9 mm, vias 0 -> 1
Changed lines of the file:
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@@
 <text x="-20.875" y="-34.993" size="1.778" layer="51" font="vector">Revised by: Brent Wilkins</text>
 <text x="19.2405" y="-9.398" size="0.8128" layer="1" font="vector" ratio="20">v01</text>
-<dimension x1="-22.098" y1="6.477" x2="22.098" y2="-6.477" x3="-30.48" y3="0" textsize="1.778" layer="20" dtype="vertical" unit="inch"/>
-<dimension x1="-18.2245" y1="-10.3505" x2="-15.031465625" y2="10.344659375" x3="-35.012628125" y3="-0.00291875" textsize="1.778" layer="20" dtype="vertical" unit="inch"/>
-<dimension x1="-22.098" y1="6.477" x2="22.098" y2="-6.477" x3="0" y3="14.683740625" textsize="1.778" layer="20" dtype="horizontal" unit="inch"/>
-<dimension x1="26.035" y1="2.54" x2="-26.035" y2="2.54" x3="0" y3="18.975325" textsize="1.778" layer="20" unit="inch"/>
-<dimension x1="22.098" y1="-6.477" x2="26.63825" y2="-11.08075" x3="28.953459375" y3="-11.0799875" textsize="1.778" layer="20" dtype="leader" unit="inch"/>
-<text x="28.991053125" y="-11.0878625" size="1.27" layer="20" font="vector">0.13" diameter typical</text>
-<text x="0" y="23.58516875" size="1.778" layer="20" font="vector" ratio="15" align="center">All units in inches</text>
+<dimension x1="-22.098" y1="6.477" x2="22.098" y2="-6.477" x3="-30.48" y3="0" textsize="1.778" layer="47" dtype="vertical" unit="inch"/>
+<dimension x1="-18.2245" y1="-10.3505" x2="-15.031465625" y2="10.344659375" x3="-35.012628125" y3="-0.00291875" textsize="1.778" layer="47" dtype="vertical" unit="inch"/>
+<dimension x1="-22.098" y1="6.477" x2="22.098" y2="-6.477" x3="0" y3="14.683740625" textsize="1.778" layer="47" dtype="horizontal" unit="inch"/>
+<dimension x1="26.035" y1="2.54" x2="-26.035" y2="2.54" x3="0" y3="18.975325" textsize="1.778" layer="47" unit="inch"/>
+<dimension x1="22.098" y1="-6.477" x2="26.63825" y2="-11.08075" x3="28.953459375" y3="-11.0799875" textsize="1.778" layer="47" dtype="leader" unit="inch"/>
+<text x="28.991053125" y="-11.0878625" size="1.27" layer="47" font="vector">0.13" diameter typical</text>
+<text x="0" y="23.58516875" size="1.778" layer="47" font="vector" ratio="15" align="center">All units in inches</text>
 <text x="23.3242625" y="0.001940625" size="1.016" layer="22" font="vector" ratio="15" rot="MR0" align="center-left">GND</text>
 <text x="23.31421875" y="2.538540625" size="1.016" layer="22" font="vector" ratio="15" rot="MR0" align="center-left">+VS</text>
@@
 <contactref element="BAT1" pad="1"/>
 <contactref element="JP2" pad="1"/>
-<wire x1="-22.43" y1="-1.498" x2="-21.183" y2="-1.498" width="0.4064" layer="1"/>
-<wire x1="-21.183" y1="-1.498" x2="-11.176" y2="8.509" width="0.4064" layer="1"/>
-<wire x1="-11.176" y1="8.509" x2="15.494" y2="8.509" width="0.4064" layer="1"/>
-<wire x1="15.494" y1="8.509" x2="20.447" y2="3.556" width="0.4064" layer="1"/>
-<wire x1="20.447" y1="3.556" x2="20.447" y2="2.159" width="0.4064" layer="1"/>
-<wire x1="20.447" y1="2.159" x2="21.108" y2="1.498" width="0.4064" layer="1"/>
-<wire x1="21.108" y1="1.498" x2="22.43" y2="1.498" width="0.4064" layer="1"/>
 <wire x1="22.43" y1="1.498" x2="23.5325" y2="1.498" width="0.4064" layer="1"/>
 <wire x1="23.5325" y1="1.498" x2="24.5745" y2="2.54" width="0.4064" layer="1"/>
+<wire x1="-22.43" y1="-1.498" x2="-22.43" y2="1.27" width="0.4064" layer="1"/>
+<via x="-22.43" y="1.27" extent="1-16" drill="0.6" shape="square"/>
+<wire x1="-22.43" y1="1.27" x2="-21.16" y2="2.54" width="0.4064" layer="16"/>
+<wire x1="-21.16" y1="2.54" x2="24.5745" y2="2.54" width="0.4064" layer="16"/>
 </signal>
 </signals>

Commit message: Moved fiducials & removed a tiny dimension layer artifact
Parts:
- moved FID1 4.02 mm to (-22.9, -7.62)
- moved FID2 4.02 mm to (22.9, 7.62)
Other:
- board size 52.1 x 20.8 mm -> 52.1 x 20.7 mm

Commit message: moved position of labeled net in schematic
Parts:
- JP1: value Power -> RAW
- JP2: value Power -> PROCESSED
Changed lines of the file:
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@@
 <layer number="113" name="IDFDebug" color="4" fill="1" visible="yes" active="yes"/>
 <layer number="116" name="Patch_BOT" color="9" fill="4" visible="yes" active="yes"/>
+<layer number="118" name="Rect_Pads" color="7" fill="1" visible="yes" active="yes"/>
 <layer number="121" name="_tsilk" color="7" fill="1" visible="yes" active="yes"/>
 <layer number="122" name="_bsilk" color="7" fill="1" visible="yes" active="yes"/>
@@
 <element name="U$5" library="advancer-technologies" package="PB-FREE" value="" x="-16.70685" y="-9.11225" rot="MR0"/>
 <element name="U$3" library="advancer-technologies" package="ROHS" value="" x="18.51025" y="-8.66775" smashed="yes" rot="MR0"/>
-<element name="JP2" library="SparkFun-Connectors" package="1X03_NO_SILK" value="Power" x="24.5745" y="2.54" smashed="yes" rot="R270"/>
+<element name="JP2" library="SparkFun-Connectors" package="1X03_NO_SILK" value="PROCESSED" x="24.5745" y="2.54" smashed="yes" rot="R270"/>
 <element name="JP3" library="SparkFunJan2012" package="STAND-OFF" value="STAND-OFF" x="22.098" y="-6.477"/>
 <element name="JP4" library="SparkFunJan2012" package="STAND-OFF" value="STAND-OFF" x="-22.098" y="6.477"/>
@@
 </element>
 <element name="U$2" library="advancer-technologies" package="ADVANCER_LOGO" value="" x="-12.954" y="6.985"/>
-<element name="JP1" library="SparkFun-Connectors" package="1X03_NO_SILK" value="Power" x="-24.5745" y="2.54" rot="R270"/>
+<element name="JP1" library="SparkFun-Connectors" package="1X03_NO_SILK" value="RAW" x="-24.5745" y="2.54" rot="R270"/>
 <element name="U$1" library="advancer-technologies" package="MYOWARE_LOGO" value="" x="0" y="0" rot="MR0"/>
 <element name="FRAME1" library="SparkFun-Aesthetics" package="CREATIVE_COMMONS" value="FRAME-LETTER" x="-32.2415" y="-32.326"/>
@@
 <contactref element="BAT1" pad="2"/>
 <contactref element="BAT2" pad="2"/>
-<contactref element="JP1" pad="3"/>
 <via x="-4.22275" y="-2.50825" extent="1-16" drill="0.508"/>
 <via x="-20.03425" y="9.17575" extent="1-16" drill="0.508"/>
 <via x="20.54225" y="9.04875" extent="1-16" drill="0.508"/>
 <via x="4.38725" y="-2.51825" extent="1-16" drill="0.508"/>
+<contactref element="JP1" pad="3"/>
 </signal>
 <signal name="SIG">
@@
 <signal name="SHLD">
 <contactref element="JP1" pad="2"/>
-</signal>
-<signal name="RAW">
-<contactref element="JP1" pad="1"/>
 </signal>
 <signal name="N$3">
@@
 <wire x1="-21.16" y1="2.54" x2="24.5745" y2="2.54" width="0.4064" layer="16"/>
 </signal>
+<signal name="RAW">
+<contactref element="JP1" pad="1"/>
+</signal>
 </signals>

Commit message: Removed RoHS claim & bumped to v10
Parts:
- removed U$3: (no value), advancer-technologies:ROHS
- removed U$5: (no value), advancer-technologies:PB-FREE
Other:
- board text added: "v10"
- board text removed: "v01"
Changed lines of the file:
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@@
 <?xml version="1.0" encoding="utf-8"?>
 <!DOCTYPE eagle SYSTEM "eagle.dtd">
-<eagle version="7.3.1">
+<eagle version="7.4.0">
 <drawing>
 <settings>
@@
 <text x="-1.825" y="-32.453" size="1.778" layer="51" font="vector">Brian E Kaminski of Advancer Technologies</text>
 <text x="-20.875" y="-34.993" size="1.778" layer="51" font="vector">Revised by: Brent Wilkins</text>
-<text x="19.2405" y="-9.398" size="0.8128" layer="1" font="vector" ratio="20">v01</text>
+<text x="18.1405" y="-9.598" size="0.8128" layer="1" font="vector" ratio="20">v10</text>
 <dimension x1="-22.098" y1="6.477" x2="22.098" y2="-6.477" x3="-30.48" y3="0" textsize="1.778" layer="47" dtype="vertical" unit="inch"/>
 <dimension x1="-18.2245" y1="-10.3505" x2="-15.031465625" y2="10.344659375" x3="-35.012628125" y3="-0.00291875" textsize="1.778" layer="47" dtype="vertical" unit="inch"/>
@@
 </autorouter>
 <elements>
-<element name="U$5" library="advancer-technologies" package="PB-FREE" value="" x="-16.70685" y="-9.11225" rot="MR0"/>
-<element name="U$3" library="advancer-technologies" package="ROHS" value="" x="18.51025" y="-8.66775" smashed="yes" rot="MR0"/>
 <element name="JP2" library="SparkFun-Connectors" package="1X03_NO_SILK" value="PROCESSED" x="24.5745" y="2.54" smashed="yes" rot="R270"/>
 <element name="JP3" library="SparkFunJan2012" package="STAND-OFF" value="STAND-OFF" x="22.098" y="-6.477"/>
