File: Hardware/MyoWare_Power_Shield.sch (EAGLE design)
At the start: 11 parts

Commit message: Updated DRC to 25mil mask limit to tent via
Other:
- note added: "v11"
- note removed: "v10"
Changed lines of the file:
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@@
 <?xml version="1.0" encoding="utf-8"?>
 <!DOCTYPE eagle SYSTEM "eagle.dtd">
-<eagle version="7.4.0">
+<eagle version="7.5.0">
 <drawing>
 <settings>
@@
 <text x="308.356" y="-46.99" size="2.54" layer="94">Brian E Kaminski of Advancer Technologies</text>
 <text x="290.83" y="-51.054" size="2.54" layer="94" ratio="10">Revised by: Brent Wilkins</text>
-<text x="378.46" y="-50.8" size="2.54" layer="94" font="vector">v10</text>
+<text x="378.46" y="-50.8" size="2.54" layer="94" font="vector">v11</text>
 <text x="261.62" y="27.94" size="1.778" layer="97" font="vector" ratio="15" align="center">VCC (+VS) +2.7V to +5.9V
 EXPECT UP TO VCC ON SIGNAL LINES</text>
